Commit message: Prva promjena

File: morus_description/urdf/morus.gazebo.xacro (robot description, xacro)
@@ -17,4 +17,5 @@
   <xacro:include filename="$(find morus_description)/urdf/morus.urdf.xacro" />
   <xacro:include filename="$(find rotors_description)/urdf/component_snippets.xacro" />
+libgazebo_ros_camera
  <!-- Mount an IMU-->
   <gazebo>
@@ -38,4 +39,22 @@
     </plugin>
   </gazebo>
+    <plugin name="lifting_surface" filename="libLiftDragPlugin.so">
+        <a0>0.08727</a0>
+        <alpha_stall>0.3368</alpha_stall>
+        <cla>5.418</cla>
+        <cla_stall>-2.1419</cla_stall>
+        <cda>0.0</cda>
+        <cda_stall>0.0</cda_stall>
+        <cma>0.0</cma>
+        <cma_stall>0.0</cma_stall>
+        <area>3</area>
+        <fluid_density>1.2041</fluid_density>
+        <forward>-1 0 0</forward>
+        <upward>0 -1 0</upward>
+        <cp>0 0 1</cp>
+        <link_name>lifting_surface_link</link_name>
+        <radial_symmetry>false</radial_symmetry>
+      </plugin>
+  <gazebo>
   <!-- Start publishing battery status msgs-->
   <gazebo>
@@ -47,5 +66,5 @@
     <plugin filename="libmorus_gazebo_battery_status.so" name="battery_status_12">
       <batteryID> 12 </batteryID>
-    </plugin>
+    </plugin>libgazebo_ros_camera
   </gazebo>
   <gazebo>
@@ -54,5 +73,5 @@
     </plugin>
   </gazebo>
-  <gazebo>
+  <gazebo>libgazebo_ros_camera
     <plugin filename="libmorus_gazebo_battery_status.so" name="battery_status_14">
       <batteryID> 14 </batteryID>

File: morus_description/urdf/morus.urdf.xacro (robot description, xacro)
@@ -20,9 +20,11 @@
   <xacro:property name="rotor_drag_coefficient" value="8.06428e-04" />
   <xacro:property name="rolling_moment_coefficient" value="0.00001" />
-  <xacro:property name="movable_mass_mass" value="1" />
-  <xacro:property name="movable_mass_dimension" value="0.08" />
-  <xacro:property name="movable_mass_offset" value="0.025" />
   <xacro:property name="imu_mass" value="0.02"/>
   <xacro:property name="imu_size" value="0.01"/>
+  <!--definirane vrijednosti za krilo -->
+  <xacro:property name="wing_mass" value="0.02"/>
+  <xacro:property name="wing_x" value="0.01"/>
+  <xacro:property name="wing_y" value="0.9"/>
+  <xacro:property name="wing_z" value="0.25"/>
   <xacro:property name="sin45" value="0.7071" />
   <xacro:property name="cos45" value="0.7071" />
@@ -40,13 +42,4 @@
     ixy="0.0" ixz="0.0"  iyz="0.0" /> <!-- [kg*m^2] [kg*m^2] [kg*m^2] [kg*m^2] [kg*m^2] [kg*m^2] -->
   </xacro:property>
-  <!-- inertia of a movable mass, assuming it is a cube. The formula is I=ms^2/6 where "s" is length of one side
-   of the cube and "m" is its mass-->
-  <xacro:property name="movable_mass_inertia">
-     <inertia
-     ixx="${(movable_mass_mass * movable_mass_dimension * movable_mass_dimension)/6}"
-     iyy="${(movable_mass_mass * movable_mass_dimension * movable_mass_dimension)/6}"
-     izz="${(movable_mass_mass * movable_mass_dimension * movable_mass_dimension)/6}"
-     ixy="0.0" ixz="0.0"  iyz="0.0" /> <!-- [kg*m^2] [kg*m^2] [kg*m^2] [kg*m^2] [kg*m^2] [kg*m^2] -->
-  </xacro:property>
   <xacro:property name="imu_inertia">
     <inertia
@@ -54,4 +47,12 @@
     iyy="${(imu_mass * imu_size * imu_size)/6}"
     izz="${(imu_mass * imu_size * imu_size)/6}"
+    ixy="0.0" ixz="0.0"  iyz="0.0" /> <!-- [kg*m^2] [kg*m^2] [kg*m^2] [kg*m^2] [kg*m^2] [kg*m^2] -->
+  </xacro:property>
+  <!-- definirana inercija za krilo -->
+  <xacro:property name="wing_inertia">
+    <inertia
+    ixx="${(wing_mass * wing_x * wing_x)/6}"
+    iyy="${(wing_mass * wing_y * wing_y)/6}"
+    izz="${(wing_mass * wing_z * wing_z)/6}"
     ixy="0.0" ixz="0.0"  iyz="0.0" /> <!-- [kg*m^2] [kg*m^2] [kg*m^2] [kg*m^2] [kg*m^2] [kg*m^2] -->
   </xacro:property>
@@ -68,4 +69,34 @@
     <xacro:insert_block name="body_inertia" />
   </xacro:multirotor_base_macro>
+  <!-- Instantiate wing_macros -->
+  <xacro:wing_macro
+    robot_namespace="$(arg name)"
+    parent="base_link"
+    wing_number="0"
+    body_width="${body_width}"
+    body_height="${body_height}"
+    mass="${wing_mass}"
+    wing_x="${wing_x}"
+    wing_y="${wing_y}"
+    wing_z="${wing_z}"
+    orientation="1">
+    <origin xyz="${body_width/2} ${body_width/2} ${body_height/2}" rpy="0 0 1.57/2" />
+    <xacro:insert_block name="wing_inertia"/>
+  </xacro:wing_macro>
+  <xacro:wing_macro
+    robot_namespace="$(arg name)"
+    parent="base_link"
+    wing_number="1"
+    body_width="${body_width}"
+    body_height="${body_height}"
+    mass="${wing_mass}"
+    wing_x="${wing_x}"
+    wing_y="${wing_y}"
+    wing_z="${wing_z}"
+    orientation="-1">
+    <origin xyz="${(-1)*body_width/2} ${(-1)*body_width/2} ${body_height/2}" rpy="0 0 1.57/2" />
+    <!-- origin xyz="0.5 0.5 0.5 " rpy="0 0 0 " -->
+    <xacro:insert_block name="wing_inertia"/>
+  </xacro:wing_macro>
   <!-- Instantiate rotors -->
   <xacro:vertical_rotor
@@ -141,76 +172,4 @@
     <xacro:insert_block name="rotor_inertia" />
   </xacro:vertical_rotor>
-  <!-- Instantiate movable mass 0-->
-  <xacro:movable_mass
-    mass_number="0"
-    parent="base_link"
-    mass="${movable_mass_mass}"
-    dimension="${movable_mass_dimension}"
-    color="Red"
-    x_axis="1"
-    y_axis="0"
-    z_axis="0"
-    orientation="${PI}">
-    <origin xyz="${(arm_length/2+arm_offset)} 0.0 ${movable_mass_offset}" rpy="0 0 0" />
-    <xacro:insert_block name="movable_mass_inertia"/>
-  </xacro:movable_mass>
-  <!-- Instantiate movable mass 1 -->
-  <xacro:movable_mass
-    mass_number="1"
-    parent="base_link"
-    mass="${movable_mass_mass}"
-    dimension="${movable_mass_dimension}"
-    color="Blue"
-    x_axis="0"
-    y_axis="1"
-    z_axis="0"
-    orientation="${PI/2}">
-    <origin xyz="0.0 ${(arm_length/2+arm_offset)} ${movable_mass_offset}" rpy="0 0 0" />
-    <xacro:insert_block name="movable_mass_inertia"/>
-  </xacro:movable_mass>
-  <!-- Instantiate movable mass 2-->
-  <xacro:movable_mass
-    mass_number="2"
-    parent="base_link"
-    mass="${movable_mass_mass}"
-    dimension="${movable_mass_dimension}"
-    color="Blue"
-    x_axis="-1"
-    y_axis="0"
-    z_axis="0"
-    orientation="${PI}">>
-    <origin xyz="${-(arm_length/2+arm_offset)} 0.0 ${movable_mass_offset}" rpy="0 0 0" />
-    <xacro:insert_block name="movable_mass_inertia"/>
-  </xacro:movable_mass>
-  <!-- Instantiate movable mass 3 -->
-  <xacro:movable_mass
-    mass_number="3"
-    parent="base_link"
-    mass="${movable_mass_mass}"
-    dimension="${movable_mass_dimension}"
-    color="Blue"
-    x_axis="0"
-    y_axis="-1"
-    z_axis="0"
-    orientation="${PI/2}">>
-    <origin xyz="0.0 ${-(arm_length/2+arm_offset)} ${movable_mass_offset}" rpy="0 0 0" />
-    <xacro:insert_block name="movable_mass_inertia"/>
-  </xacro:movable_mass>
-  <xacro:transmisija
-    trans_number="0"
-    joint_name="stick_to_movable_mass_0">
-  </xacro:transmisija>
-  <xacro:transmisija
-    trans_number="1"
-    joint_name="stick_to_movable_mass_1">
-  </xacro:transmisija>
-  <xacro:transmisija
-    trans_number="2"
-    joint_name="stick_to_movable_mass_2">
-  </xacro:transmisija>
-  <xacro:transmisija
-    trans_number="3"
-    joint_name="stick_to_movable_mass_3">
-  </xacro:transmisija>
   <xacro:property name="land_gear_inertia">
     <inertia

File: morus_description/urdf/multirotor_base.urdf.xacro (robot description, xacro)
@@ -56,41 +56,32 @@
     </gazebo>
   </xacro:macro>
-  <!-- Macro file for movable mass. It defines joint between mass and stick, and link which defines actual mass. Stick
-  is defined in other macro file-->
-  <xacro:macro name="movable_mass" params="mass_number parent mass dimension color x_axis y_axis z_axis orientation *origin *inertia">
-    <joint name="stick_to_movable_mass_${mass_number}" type="prismatic">
-      <xacro:insert_block name="origin"/>
-      <axis xyz="${x_axis} ${y_axis} ${z_axis}"/>
+  <!-- Macro file for wing. It defines joint between base and wing.-->
+  <xacro:macro name="wing_macro"
+     params="robot_namespace parent wing_number body_width body_height mass wing_x wing_y wing_z  orientation *origin *inertia">
+    <joint name="base_to_wing_${wing_number}" type="fixed">
+    <xacro:insert_block name="origin" />
+      <axis xyz="0 0 0"/>
       <parent link="${parent}"/>
-      <child link="movable_mass_${mass_number}"/>
-      <limit lower="-0.3" upper="0.3" effort="10000" velocity="20"/>
-      <dynamics damping="10" />  <!--friction="0.1" used only in Gazebo >= 5.0, damping is the viscous friction damping,
-       i.e. Ft = damping * v -->
-    </joint>
-    <link name="movable_mass_${mass_number}">
-      <visual>
-        <!--origin rpy="0 0 ${orientation}" xyz="0 0 ${0*movable_mass_dimension/2}"/-->
-        <origin rpy="0 0 ${orientation}" xyz="0 0 0"/>
-        <geometry>
-          <!--mesh filename="package://morus_description/meshes/${mesh_file_mass}"
-            scale="1 1 1" /-->
-          <box size="${1*dimension} ${1*dimension} ${1*dimension}"/>
-        </geometry>
-      </visual>
-      <collision>
-        <origin rpy="0 0 0" xyz="0 0 ${0*movable_mass_dimension/2}"/>
-        <geometry>
-          <box size="${dimension} ${dimension} ${dimension}"/>
-        </geometry>
-      </collision>
-      <inertial>
-        <origin rpy="0 0 0" xyz="0 0 ${0*movable_mass_dimension/2}"/>
-        <mass value="${mass}"/>
+      <child link="wing_${wing_number}"/>
+    </joint>
+    <link name="wing_${wing_number}">
+      <visual>
+        <origin rpy="0 0 0" xyz="0 0 0"/>
+        <geometry>
+          <box size="${1*wing_x} ${1*wing_y} ${1*wing_z}"/>
+        </geometry>
+      </visual>
+      <collision>
+        <origin rpy="0 0 0" xyz="0 0 0"/>
+        <geometry>
+          <box size="${wing_x} ${wing_y} ${wing_z}"/>
+        </geometry>
+      </collision>
+      <inertial>
+        <origin rpy="0 0 0" xyz="0 0 0"/>
+        <mass value="${wing_mass}"/>
         <xacro:insert_block name="inertia"/>
       </inertial>
     </link>
-    <gazebo reference="movable_mass_${mass_number}">
-      <material>Gazebo/${color}</material>
-    </gazebo>
   </xacro:macro>
   <!-- Rotor joint and link -->

Commit message: Druga promjena

File: morus_description/urdf/morus.gazebo.xacro (robot description, xacro)
@@ -39,22 +39,4 @@
     </plugin>
   </gazebo>
-    <plugin name="lifting_surface" filename="libLiftDragPlugin.so">
-        <a0>0.08727</a0>
-        <alpha_stall>0.3368</alpha_stall>
-        <cla>5.418</cla>
-        <cla_stall>-2.1419</cla_stall>
-        <cda>0.0</cda>
-        <cda_stall>0.0</cda_stall>
-        <cma>0.0</cma>
-        <cma_stall>0.0</cma_stall>
-        <area>3</area>
-        <fluid_density>1.2041</fluid_density>
-        <forward>-1 0 0</forward>
-        <upward>0 -1 0</upward>
-        <cp>0 0 1</cp>
-        <link_name>lifting_surface_link</link_name>
-        <radial_symmetry>false</radial_symmetry>
-      </plugin>
-  <gazebo>
   <!-- Start publishing battery status msgs-->
   <gazebo>

File: morus_description/urdf/morus.urdf.xacro (robot description, xacro)
@@ -81,5 +81,5 @@
     wing_z="${wing_z}"
     orientation="1">
-    <origin xyz="${body_width/2} ${body_width/2} ${body_height/2}" rpy="0 0 1.57/2" />
+    <origin xyz="${body_width/2} ${body_width/2} ${body_height/2}" rpy="0 0 0.79" />
     <xacro:insert_block name="wing_inertia"/>
   </xacro:wing_macro>
@@ -95,5 +95,5 @@
     wing_z="${wing_z}"
     orientation="-1">
-    <origin xyz="${(-1)*body_width/2} ${(-1)*body_width/2} ${body_height/2}" rpy="0 0 1.57/2" />
+    <origin xyz="${(-1)*body_width/2} ${(-1)*body_width/2} ${body_height/2}" rpy="0 0 0.79" />
     <!-- origin xyz="0.5 0.5 0.5 " rpy="0 0 0 " -->
     <xacro:insert_block name="wing_inertia"/>

File: morus_description/urdf/multirotor_base.urdf.xacro (robot description, xacro)
@@ -84,4 +84,23 @@
       </inertial>
     </link>
+    <gazebo>
+      <plugin name="lifting_surface_${wing_number}" filename="libLiftDragPlugin.so">
+        <a0>0.08727</a0>
+        <alpha_stall>0.3368</alpha_stall>
+        <cla>5.418</cla>
+        <cla_stall>-2.1419</cla_stall>
+        <cda>0.0</cda>
+        <cda_stall>0.0</cda_stall>
+        <cma>0.0</cma>
+        <cma_stall>0.0</cma_stall>
+        <area>3</area>
+        <fluid_density>1.2041</fluid_density>
+        <forward>-1 0 0</forward>
+        <upward>0 -1 0</upward>
+        <cp>0 0 1</cp>
+        <!-- <link_name>wing_${wing_number}</link_name> -->
+        <control_joint_name>base_to_wing_${wing_number}</control_joint_name>
+      </plugin>
+    </gazebo>
   </xacro:macro>
   <!-- Rotor joint and link -->
