Commit message: Krila

File: morus_description/urdf/morus.urdf.xacro (robot description, xacro)
@@ -25,5 +25,5 @@
   <xacro:property name="wing_mass" value="0.02"/>
   <xacro:property name="wing_x" value="0.01"/>
-  <xacro:property name="wing_y" value="0.9"/>
+  <xacro:property name="wing_y" value="1.3"/>
   <xacro:property name="wing_z" value="0.25"/>
   <xacro:property name="sin45" value="0.7071" />
@@ -80,6 +80,7 @@
     wing_y="${wing_y}"
     wing_z="${wing_z}"
-    orientation="1">
-    <origin xyz="${body_width/2} ${body_width/2} ${body_height/2}" rpy="0 0 0.79" />
+    orientation="1"
+    color="Red">
+    <origin xyz="${body_width/2} ${body_width/2} 0" rpy="0 0 5.495" />
     <xacro:insert_block name="wing_inertia"/>
   </xacro:wing_macro>
@@ -94,7 +95,7 @@
     wing_y="${wing_y}"
     wing_z="${wing_z}"
-    orientation="-1">
-    <origin xyz="${(-1)*body_width/2} ${(-1)*body_width/2} ${body_height/2}" rpy="0 0 0.79" />
-    <!-- origin xyz="0.5 0.5 0.5 " rpy="0 0 0 " -->
+    orientation="1"
+    color="Blue">
+    <origin xyz="${(-1)*body_width/2} ${(-1)*body_width/2} 0" rpy="0 0 2.355" />
     <xacro:insert_block name="wing_inertia"/>
   </xacro:wing_macro>

File: morus_description/urdf/multirotor_base.urdf.xacro (robot description, xacro)
@@ -58,5 +58,5 @@
   <!-- Macro file for wing. It defines joint between base and wing.-->
   <xacro:macro name="wing_macro"
-     params="robot_namespace parent wing_number body_width body_height mass wing_x wing_y wing_z  orientation *origin *inertia">
+     params="robot_namespace parent wing_number body_width body_height mass wing_x wing_y wing_z  orientation color *origin *inertia">
     <joint name="base_to_wing_${wing_number}" type="fixed">
     <xacro:insert_block name="origin" />
@@ -67,5 +67,6 @@
     <link name="wing_${wing_number}">
       <visual>
-        <origin rpy="0 0 0" xyz="0 0 0"/>
+        <!-- <origin rpy="0 0 0" xyz="0 ${orientation*wing_y*0.5} 0"/> -->
+        <origin rpy="0 0 0" xyz="0 ${orientation*wing_y*0.5} 0"/>
         <geometry>
           <box size="${1*wing_x} ${1*wing_y} ${1*wing_z}"/>
@@ -73,5 +74,5 @@
       </visual>
       <collision>
-        <origin rpy="0 0 0" xyz="0 0 0"/>
+        <origin rpy="0 0 0" xyz="0 ${orientation*wing_y*0.5} 0"/>
         <geometry>
           <box size="${wing_x} ${wing_y} ${wing_z}"/>
@@ -79,5 +80,5 @@
       </collision>
       <inertial>
-        <origin rpy="0 0 0" xyz="0 0 0"/>
+        <origin rpy="0 0 0" xyz="0 ${orientation*wing_y*0.5} 0"/>
         <mass value="${wing_mass}"/>
         <xacro:insert_block name="inertia"/>
@@ -102,4 +103,7 @@
         <control_joint_name>base_to_wing_${wing_number}</control_joint_name>
       </plugin>
+    </gazebo>
+    <gazebo reference="wing_${wing_number}">
+      <material>Gazebo/${color}</material>
     </gazebo>
   </xacro:macro>
